File: 555_Badge/555_Badge.sch (KiCad schematic (older format))
At the start: 15 parts

Commit message: Add footprints partial
Parts:
- C1: renamed from C?; footprint (none) -> Capacitor_THT:CP_Radial_D5.0mm_P2.00mm
- gave numbers to parts that had none: 14
Changed lines of the file:
@@
 $EndDescr
 $Comp
-L 555_Badge:7555 U?
+L 555_Badge:7555 U1
 U 1 1 61238510
 P 5950 3450
-F 0 "U?" H 5600 4000 50  0000 L CNN
+F 0 "U1" H 5600 4000 50  0000 L CNN
 F 1 "7555" H 6150 2850 50  0000 L CNN
 F 2 "" H 5900 3350 50  0001 C CNN
@@
 $EndComp
 $Comp
-L Device:R R?
+L Device:R R1
 U 1 1 6124C785
 P 4400 3000
-F 0 "R?" H 4470 3046 50  0000 L CNN
+F 0 "R1" H 4470 3046 50  0000 L CNN
 F 1 "22e3" H 4470 2955 50  0000 L CNN
 F 2 "" V 4330 3000 50  0001 C CNN
@@
 $EndComp
 $Comp
-L Device:R R?
+L Device:R R2
 U 1 1 6124CF23
 P 4400 3750
-F 0 "R?" H 4470 3796 50  0000 L CNN
+F 0 "R2" H 4470 3796 50  0000 L CNN
 F 1 "330e3" H 4470 3705 50  0000 L CNN
 F 2 "" V 4330 3750 50  0001 C CNN
@@
 $EndComp
 $Comp
-L Device:R R?
+L Device:R R3
 U 1 1 6124D459
 P 7000 3650
-F 0 "R?" V 6793 3650 50  0000 C CNN
+F 0 "R3" V 6793 3650 50  0000 C CNN
 F 1 "22e3" V 6884 3650 50  0000 C CNN
 F 2 "" V 6930 3650 50  0001 C CNN
@@
 $EndComp
 $Comp
-L Device:R R?
+L Device:R R4
 U 1 1 6124DBDA
 P 7400 3950
-F 0 "R?" H 7470 3996 50  0000 L CNN
+F 0 "R4" H 7470 3996 50  0000 L CNN
 F 1 "100e3" H 7470 3905 50  0000 L CNN
 F 2 "" V 7330 3950 50  0001 C CNN
@@
 $EndComp
 $Comp
-L Device:R R?
+L Device:R R5
 U 1 1 6124E115
 P 8250 3650
-F 0 "R?" V 8043 3650 50  0000 C CNN
+F 0 "R5" V 8043 3650 50  0000 C CNN
 F 1 "10e3" V 8134 3650 50  0000 C CNN
 F 2 "" V 8180 3650 50  0001 C CNN
@@
 $EndComp
 $Comp
-L Device:R R?
+L Device:R R6
 U 1 1 6124EB36
 P 8900 2600
-F 0 "R?" H 8970 2646 50  0000 L CNN
+F 0 "R6" H 8970 2646 50  0000 L CNN
 F 1 "100" H 8970 2555 50  0000 L CNN
 F 2 "" V 8830 2600 50  0001 C CNN
@@
 $EndComp
 $Comp
-L Device:R R?
+L Device:R R7
 U 1 1 6124F0CC
 P 9300 2600
-F 0 "R?" H 9370 2646 50  0000 L CNN
+F 0 "R7" H 9370 2646 50  0000 L CNN
 F 1 "100" H 9370 2555 50  0000 L CNN
 F 2 "" V 9230 2600 50  0001 C CNN
@@
 $EndComp
 $Comp
-L Device:CP1 C?
+L Device:CP1 C1
 U 1 1 6124F635
 P 4400 4350
-F 0 "C?" H 4515 4396 50  0000 L CNN
+F 0 "C1" H 4515 4396 50  0000 L CNN
 F 1 "10e-6" H 4515 4305 50  0000 L CNN
-F 2 "" H 4400 4350 50  0001 C CNN
+F 2 "Capacitor_THT:CP_Radial_D5.0mm_P2.00mm" H 4400 4350 50  0001 C CNN
 F 3 "~" H 4400 4350 50  0001 C CNN
 	1    4400 4350
@@
 $EndComp
 $Comp
-L Device:CP1 C?
+L Device:CP1 C2
 U 1 1 6124FCB0
 P 7850 3950
-F 0 "C?" H 7965 3996 50  0000 L CNN
+F 0 "C2" H 7965 3996 50  0000 L CNN
 F 1 "100e-6" H 7965 3905 50  0000 L CNN
 F 2 "" H 7850 3950 50  0001 C CNN
@@
 $EndComp
 $Comp
-L Device:LED D?
+L Device:LED D1
 U 1 1 61252413
 P 8900 3050
-F 0 "D?" V 8939 2932 50  0000 R CNN
+F 0 "D1" V 8939 2932 50  0000 R CNN
 F 1 "RED" V 8848 2932 50  0000 R CNN
 F 2 "" H 8900 3050 50  0001 C CNN
@@
 $EndComp
 $Comp
-L Device:LED D?
+L Device:LED D2
 U 1 1 61253075
 P 9300 3050
-F 0 "D?" V 9339 2932 50  0000 R CNN
+F 0 "D2" V 9339 2932 50  0000 R CNN
 F 1 "RED" V 9248 2932 50  0000 R CNN
 F 2 "" H 9300 3050 50  0001 C CNN
@@
 $EndComp
 $Comp
-L Transistor_BJT:2N3904 Q?
+L Transistor_BJT:2N3904 Q1
 U 1 1 61253832
 P 8800 3650
-F 0 "Q?" H 8990 3696 50  0000 L CNN
+F 0 "Q1" H 8990 3696 50  0000 L CNN
 F 1 "2N3904" H 8990 3605 50  0000 L CNN
 F 2 "Package_TO_SOT_THT:TO-92_Inline" H 9000 3575 50  0001 L CIN
@@
 $EndComp
 $Comp
-L dk_Battery-Holders-Clips-Contacts:BS-7 BAT?
+L dk_Battery-Holders-Clips-Contacts:BS-7 BAT1
 U 1 1 6125515F
 P 3350 3800
-F 0 "BAT?" H 3478 3853 60  0000 L CNN
+F 0 "BAT1" H 3478 3853 60  0000 L CNN
 F 1 "BS-7" H 3478 3747 60  0000 L CNN
 F 2 "digikey-footprints:Battery_Holder_Coin_2032_BS-7" H 3550 4000 60  0001 L CNN
@@
 $EndComp
 $Comp
-L dk_Slide-Switches:EG1218 S?
+L dk_Slide-Switches:EG1218 S1
 U 1 1 61256877
 P 3450 3100
-F 0 "S?" V 3404 3244 50  0000 L CNN
+F 0 "S1" V 3404 3244 50  0000 L CNN
 F 1 "EG1218" V 3495 3244 50  0000 L CNN
 F 2 "digikey-footprints:Switch_Slide_11.6x4mm_EG1218" H 3650 3300 50  0001 L CNN
@@
 $EndComp
 $Comp
-L power:GND #PWR?
+L power:GND #PWR04
 U 1 1 6125ABDB
 P 4400 4650
-F 0 "#PWR?" H 4400 4400 50  0001 C CNN
+F 0 "#PWR04" H 4400 4400 50  0001 C CNN
 F 1 "GND" H 4405 4477 50  0000 C CNN
 F 2 "" H 4400 4650 50  0001 C CNN
@@
 $EndComp
 $Comp
-L power:GND #PWR?
+L power:GND #PWR01
 U 1 1 6125B250
 P 3350 4150
-F 0 "#PWR?" H 3350 3900 50  0001 C CNN
+F 0 "#PWR01" H 3350 3900 50  0001 C CNN
 F 1 "GND" H 3355 3977 50  0000 C CNN
 F 2 "" H 3350 4150 50  0001 C CNN
@@
 $EndComp
 $Comp
-L power:GND #PWR?
+L power:GND #PWR05
 U 1 1 6125B8E5
 P 5900 4150
-F 0 "#PWR?" H 5900 3900 50  0001 C CNN
+F 0 "#PWR05" H 5900 3900 50  0001 C CNN
 F 1 "GND" H 5905 3977 50  0000 C CNN
 F 2 "" H 5900 4150 50  0001 C CNN
@@
 $EndComp
 $Comp
-L power:GND #PWR?
+L power:GND #PWR07
 U 1 1 6125BDD6
 P 7400 4300
-F 0 "#PWR?" H 7400 4050 50  0001 C CNN
+F 0 "#PWR07" H 7400 4050 50  0001 C CNN
 F 1 "GND" H 7405 4127 50  0000 C CNN
 F 2 "" H 7400 4300 50  0001 C CNN
@@
 $EndComp
 $Comp
-L power:GND #PWR?
+L power:GND #PWR08
 U 1 1 6125C147
 P 7850 4300
-F 0 "#PWR?" H 7850 4050 50  0001 C CNN
+F 0 "#PWR08" H 7850 4050 50  0001 C CNN
 F 1 "GND" H 7855 4127 50  0000 C CNN
 F 2 "" H 7850 4300 50  0001 C CNN
@@
 $EndComp
 $Comp
-L power:GND #PWR?
+L power:GND #PWR010
 U 1 1 6125C400
 P 8900 4050
-F 0 "#PWR?" H 8900 3800 50  0001 C CNN
+F 0 "#PWR010" H 8900 3800 50  0001 C CNN
 F 1 "GND" H 8905 3877 50  0000 C CNN
 F 2 "" H 8900 4050 50  0001 C CNN
@@
 $EndComp
 $Comp
-L power:VCC #PWR?
+L power:VCC #PWR02
 U 1 1 6125CC56
 P 3450 2700
-F 0 "#PWR?" H 3450 2550 50  0001 C CNN
+F 0 "#PWR02" H 3450 2550 50  0001 C CNN
 F 1 "VCC" H 3465 2873 50  0000 C CNN
 F 2 "" H 3450 2700 50  0001 C CNN
@@
 $EndComp
 $Comp
-L power:VCC #PWR?
+L power:VCC #PWR06
 U 1 1 6127689E
 P 6100 2700
-F 0 "#PWR?" H 6100 2550 50  0001 C CNN
+F 0 "#PWR06" H 6100 2550 50  0001 C CNN
 F 1 "VCC" H 6115 2873 50  0000 C CNN
 F 2 "" H 6100 2700 50  0001 C CNN
@@
 $EndComp
 $Comp
-L power:VCC #PWR?
+L power:VCC #PWR03
 U 1 1 61276FB8
 P 4400 2700
-F 0 "#PWR?" H 4400 2550 50  0001 C CNN
+F 0 "#PWR03" H 4400 2550 50  0001 C CNN
 F 1 "VCC" H 4415 2873 50  0000 C CNN
 F 2 "" H 4400 2700 50  0001 C CNN
@@
 $EndComp
 $Comp
-L power:VCC #PWR?
+L power:VCC #PWR09
 U 1 1 6127754F
 P 8900 2300
-F 0 "#PWR?" H 8900 2150 50  0001 C CNN
+F 0 "#PWR09" H 8900 2150 50  0001 C CNN
 F 1 "VCC" H 8915 2473 50  0000 C CNN
 F 2 "" H 8900 2300 50  0001 C CNN
@@
 $EndComp
 $Comp
-L power:VCC #PWR?
+L power:VCC #PWR011
 U 1 1 61277B59
 P 9300 2300
-F 0 "#PWR?" H 9300 2150 50  0001 C CNN
+F 0 "#PWR011" H 9300 2150 50  0001 C CNN
 F 1 "VCC" H 9315 2473 50  0000 C CNN
 F 2 "" H 9300 2300 50  0001 C CNN

Commit message: Add footprints complete
Parts:
- C2: footprint (none) -> Capacitor_THT:CP_Radial_D6.3mm_P2.50mm
- D1, D2: footprint (none) -> LED_THT:LED_D3.0mm
- R1, R2, R3, R4, R5, R6, R7: footprint (none) -> Resistor_THT:R_Axial_DIN0207_L6.3mm_D2.5mm_P7.62mm_Horizontal
- U1: footprint (none) -> 555_Badge:ICM7555-PDIP
Changed lines of the file:
@@
 F 0 "U1" H 5600 4000 50  0000 L CNN
 F 1 "7555" H 6150 2850 50  0000 L CNN
-F 2 "" H 5900 3350 50  0001 C CNN
+F 2 "555_Badge:ICM7555-PDIP" H 5900 3350 50  0001 C CNN
 F 3 "https://www.renesas.com/us/en/document/dst/icm7555-icm7556-datasheet" H 5900 3350 50  0001 C CNN
 	1    5950 3450
@@
 F 0 "R1" H 4470 3046 50  0000 L CNN
 F 1 "22e3" H 4470 2955 50  0000 L CNN
-F 2 "" V 4330 3000 50  0001 C CNN
+F 2 "Resistor_THT:R_Axial_DIN0207_L6.3mm_D2.5mm_P7.62mm_Horizontal" V 4330 3000 50  0001 C CNN
 F 3 "~" H 4400 3000 50  0001 C CNN
 	1    4400 3000
@@
 F 0 "R2" H 4470 3796 50  0000 L CNN
 F 1 "330e3" H 4470 3705 50  0000 L CNN
-F 2 "" V 4330 3750 50  0001 C CNN
+F 2 "Resistor_THT:R_Axial_DIN0207_L6.3mm_D2.5mm_P7.62mm_Horizontal" V 4330 3750 50  0001 C CNN
 F 3 "~" H 4400 3750 50  0001 C CNN
 	1    4400 3750
@@
 F 0 "R3" V 6793 3650 50  0000 C CNN
 F 1 "22e3" V 6884 3650 50  0000 C CNN
-F 2 "" V 6930 3650 50  0001 C CNN
+F 2 "Resistor_THT:R_Axial_DIN0207_L6.3mm_D2.5mm_P7.62mm_Horizontal" V 6930 3650 50  0001 C CNN
 F 3 "~" H 7000 3650 50  0001 C CNN
 	1    7000 3650
@@
 F 0 "R4" H 7470 3996 50  0000 L CNN
 F 1 "100e3" H 7470 3905 50  0000 L CNN
-F 2 "" V 7330 3950 50  0001 C CNN
+F 2 "Resistor_THT:R_Axial_DIN0207_L6.3mm_D2.5mm_P7.62mm_Horizontal" V 7330 3950 50  0001 C CNN
 F 3 "~" H 7400 3950 50  0001 C CNN
 	1    7400 3950
@@
 F 0 "R5" V 8043 3650 50  0000 C CNN
 F 1 "10e3" V 8134 3650 50  0000 C CNN
-F 2 "" V 8180 3650 50  0001 C CNN
+F 2 "Resistor_THT:R_Axial_DIN0207_L6.3mm_D2.5mm_P7.62mm_Horizontal" V 8180 3650 50  0001 C CNN
 F 3 "~" H 8250 3650 50  0001 C CNN
 	1    8250 3650
@@
 F 0 "R6" H 8970 2646 50  0000 L CNN
 F 1 "100" H 8970 2555 50  0000 L CNN
-F 2 "" V 8830 2600 50  0001 C CNN
+F 2 "Resistor_THT:R_Axial_DIN0207_L6.3mm_D2.5mm_P7.62mm_Horizontal" V 8830 2600 50  0001 C CNN
 F 3 "~" H 8900 2600 50  0001 C CNN
 	1    8900 2600
@@
 F 0 "R7" H 9370 2646 50  0000 L CNN
 F 1 "100" H 9370 2555 50  0000 L CNN
-F 2 "" V 9230 2600 50  0001 C CNN
+F 2 "Resistor_THT:R_Axial_DIN0207_L6.3mm_D2.5mm_P7.62mm_Horizontal" V 9230 2600 50  0001 C CNN
 F 3 "~" H 9300 2600 50  0001 C CNN
 	1    9300 2600
@@
 F 0 "C2" H 7965 3996 50  0000 L CNN
 F 1 "100e-6" H 7965 3905 50  0000 L CNN
-F 2 "" H 7850 3950 50  0001 C CNN
+F 2 "Capacitor_THT:CP_Radial_D6.3mm_P2.50mm" H 7850 3950 50  0001 C CNN
 F 3 "~" H 7850 3950 50  0001 C CNN
 	1    7850 3950
@@
 F 0 "D1" V 8939 2932 50  0000 R CNN
 F 1 "RED" V 8848 2932 50  0000 R CNN
-F 2 "" H 8900 3050 50  0001 C CNN
+F 2 "LED_THT:LED_D3.0mm" H 8900 3050 50  0001 C CNN
 F 3 "~" H 8900 3050 50  0001 C CNN
 	1    8900 3050
@@
 F 0 "D2" V 9339 2932 50  0000 R CNN
 F 1 "RED" V 9248 2932 50  0000 R CNN
-F 2 "" H 9300 3050 50  0001 C CNN
+F 2 "LED_THT:LED_D3.0mm" H 9300 3050 50  0001 C CNN
 F 3 "~" H 9300 3050 50  0001 C CNN
 	1    9300 3050
